File: kicad/mmx-vrm.kicad_pcb (KiCad board)
At the start: 2 copper layers, 39.8 x 43.9 mm, 18 parts, among them J1 Conn_02x15_Row_Letter_First, SW1 SW_DIP_x03, U1 LM2596S, U2 LM2596S

Commit message: Resistors annotation renumber
Parts:
- R1: renamed from F1; value Fuse -> 0
- renumbered R3 to R2, R4 to R3, R5 to R4, R6 to R5, R7 to R6, R8 to R7
