File: kicad/mmx-vrm.sch (KiCad schematic (older format))
At the start: 17 parts, among them J1 Conn_02x15_Row_Letter_First, SW1 SW_DIP_x03, U1 LM2596S, U2 LM2596S

Commit message: Resistors annotation renumber
Parts:
- R1: renamed from F1; value Fuse -> 0; symbol Device:Fuse -> Device:R
- renumbered R3 to R2, R4 to R3, R5 to R4, R6 to R5, R7 to R6, R8 to R7
Changed lines of the file:
@@
 	2600 3800 2850 3800
 $Comp
-L Device:R R8
+L Device:R R7
 U 1 1 60E41091
 P 7000 3500
-F 0 "R8" H 7050 3550 50  0000 L CNN
+F 0 "R7" H 7050 3550 50  0000 L CNN
 F 1 "1K" V 7000 3450 50  0000 L CNN
 F 2 "Resistor_SMD:R_1206_3216Metric_Pad1.30x1.75mm_HandSolder" V 6930 3500 50  0001 C CNN
@@
 $EndComp
 $Comp
-L Device:R R7
+L Device:R R6
 U 1 1 60E4143A
 P 7250 2500
-F 0 "R7" H 7300 2550 50  0000 L CNN
+F 0 "R6" H 7300 2550 50  0000 L CNN
 F 1 "1.5K" V 7250 2400 50  0000 L CNN
 F 2 "Resistor_SMD:R_1206_3216Metric_Pad1.30x1.75mm_HandSolder" V 7180 2500 50  0001 C CNN
@@
 	7250 2650 7250 3350
 $Comp
-L Device:R R6
+L Device:R R5
 U 1 1 60E59BB7
 P 7100 2500
-F 0 "R6" H 7050 2700 50  0000 L CNN
+F 0 "R5" H 7050 2700 50  0000 L CNN
 F 1 "3K" V 7100 2450 50  0000 L CNN
 F 2 "Resistor_SMD:R_1206_3216Metric_Pad1.30x1.75mm_HandSolder" V 7030 2500 50  0001 C CNN
@@
 	6900 2350 7000 2350
 $Comp
-L Device:R R4
+L Device:R R3
 U 1 1 60E5A2A0
 P 6900 2500
-F 0 "R4" H 6850 2700 50  0000 L CNN
+F 0 "R3" H 6850 2700 50  0000 L CNN
 F 1 "15K" V 6900 2400 50  0000 L CNN
 F 2 "Resistor_SMD:R_1206_3216Metric_Pad1.30x1.75mm_HandSolder" V 6830 2500 50  0001 C CNN
@@
 $EndComp
 $Comp
-L Device:R R5
+L Device:R R4
 U 1 1 60E59F40
 P 7000 2500
-F 0 "R5" H 6950 2700 50  0000 L CNN
+F 0 "R4" H 6950 2700 50  0000 L CNN
 F 1 "7.5K" V 7000 2400 50  0000 L CNN
 F 2 "Resistor_SMD:R_1206_3216Metric_Pad1.30x1.75mm_HandSolder" V 6930 2500 50  0001 C CNN
@@
 $EndComp
 $Comp
-L Device:R R3
+L Device:R R2
 U 1 1 60E7644A
 P 7650 2800
-F 0 "R3" V 7750 2800 50  0000 C CNN
+F 0 "R2" V 7750 2800 50  0000 C CNN
 F 1 "1K" V 7650 2800 50  0000 C CNN
 F 2 "Resistor_SMD:R_1206_3216Metric_Pad1.30x1.75mm_HandSolder" V 7580 2800 50  0001 C CNN
@@
 VCORE
 $Comp
-L Device:Fuse F1
+L Device:R R1
 U 1 1 612477AD
 P 2700 4100
-F 0 "F1" V 2600 4100 50  0000 C CNN
-F 1 "Fuse" V 2800 4100 50  0000 C CNN
+F 0 "R1" V 2600 4100 50  0000 C CNN
+F 1 "0" V 2700 4100 50  0000 C CNN
 F 2 "Resistor_SMD:R_1206_3216Metric_Pad1.30x1.75mm_HandSolder" V 2630 4100 50  0001 C CNN
 F 3 "~" H 2700 4100 50  0001 C CNN

Commit message: LCSC number for the voltage regulator
Parts:
- U1, U2: LCSC C74191 -> C74188
Changed lines of the file:
@@
 F 2 "Package_TO_SOT_SMD:TO-263-5_TabPin3" H 5100 2000 50  0001 L CIN
 F 3 "http://www.ti.com/lit/ds/symlink/lm2596.pdf" H 5050 2250 50  0001 C CNN
-F 4 "C74191" H 5050 2250 50  0001 C CNN "LCSC"
+F 4 "C74188" H 5050 2250 50  0001 C CNN "LCSC"
 	1    5050 2250
 	1    0    0    -1
@@
 F 2 "Package_TO_SOT_SMD:TO-263-5_TabPin3" H 5050 3200 50  0001 L CIN
 F 3 "http://www.ti.com/lit/ds/symlink/lm2596.pdf" H 5000 3450 50  0001 C CNN
-F 4 "C74191" H 5000 3450 50  0001 C CNN "LCSC"
+F 4 "C74188" H 5000 3450 50  0001 C CNN "LCSC"
 	1    5000 3450
 	1    0    0    -1

Commit message: Fixes after first tests
Parts:
- added C3: 10nF, Capacitor_SMD:C_1206_3216Metric_Pad1.33x1.80mm_HandSolder, symbol Device:C
Connections:
- wire segments 44 -> 48
Changed lines of the file:
@@
 Sheet 1 1
 Title "MMX-VRM"
-Date "2021-09-06"
+Date "2021-11-16"
 Rev "0.2"
 Comp "Necroware"
@@
 Connection ~ 6450 2350
 Wire Wire Line
-	6450 2350 6900 2350
+	6450 2350 6600 2350
 Connection ~ 4000 2150
 Wire Wire Line
@@
 Connection ~ 6250 3350
 Wire Wire Line
-	6250 3350 6900 3350
+	6250 3350 6600 3350
 Wire Wire Line
 	7500 2350 7500 2800
@@
 	0    1    1    0
 $EndComp
+$Comp
+L Device:C C3
+U 1 1 6192E569
+P 6600 2650
+F 0 "C3" H 6600 2750 50  0000 L CNN
+F 1 "10nF" H 6600 2550 50  0000 L CNN
+F 2 "Capacitor_SMD:C_1206_3216Metric_Pad1.33x1.80mm_HandSolder" H 6638 2500 50  0001 C CNN
+F 3 "~" H 6600 2650 50  0001 C CNN
+F 4 "C431006" H 6600 2650 50  0001 C CNN "LCSC"
+	1    6600 2650
+	1    0    0    -1
+$EndComp
+Wire Wire Line
+	6600 2350 6600 2500
+Connection ~ 6600 2350
+Wire Wire Line
+	6600 2350 6900 2350
+Wire Wire Line
+	6600 2800 6600 3350
+Connection ~ 6600 3350
+Wire Wire Line
+	6600 3350 6900 3350
 $EndSCHEMATC

Commit message: Readjusted the resistors for 3.2V support
Parts:
- R3: value 15K -> 9K; LCSC C319849 -> C488999
- R4: value 7.5K -> 6.3K; LCSC C352034 -> C488915
- R5: value 3K -> 2.9K; LCSC C18012 -> C488724
- R6: value 1.5K -> 1.6K; LCSC C26030 -> C204679
Changed lines of the file:
@@
 Sheet 1 1
 Title "MMX-VRM"
-Date "2021-11-16"
+Date "2021-11-19"
 Rev "0.2"
 Comp "Necroware"
@@
 P 7250 2500
 F 0 "R6" H 7300 2550 50  0000 L CNN
-F 1 "1.5K" V 7250 2400 50  0000 L CNN
+F 1 "1.6K" V 7250 2400 50  0000 L CNN
 F 2 "Resistor_SMD:R_1206_3216Metric_Pad1.30x1.75mm_HandSolder" V 7180 2500 50  0001 C CNN
 F 3 "~" H 7250 2500 50  0001 C CNN
-F 4 "C26030" H 7250 2500 50  0001 C CNN "LCSC"
+F 4 "C204679" H 7250 2500 50  0001 C CNN "LCSC"
 	1    7250 2500
 	1    0    0    -1
@@
 P 7100 2500
 F 0 "R5" H 7050 2700 50  0000 L CNN
-F 1 "3K" V 7100 2450 50  0000 L CNN
+F 1 "2.9K" V 7100 2450 50  0000 L CNN
 F 2 "Resistor_SMD:R_1206_3216Metric_Pad1.30x1.75mm_HandSolder" V 7030 2500 50  0001 C CNN
 F 3 "~" H 7100 2500 50  0001 C CNN
-F 4 "C18012" H 7100 2500 50  0001 C CNN "LCSC"
+F 4 "C488724" H 7100 2500 50  0001 C CNN "LCSC"
 	1    7100 2500
 	1    0    0    -1
@@
 P 6900 2500
 F 0 "R3" H 6850 2700 50  0000 L CNN
-F 1 "15K" V 6900 2400 50  0000 L CNN
+F 1 "9K" V 6900 2400 50  0000 L CNN
 F 2 "Resistor_SMD:R_1206_3216Metric_Pad1.30x1.75mm_HandSolder" V 6830 2500 50  0001 C CNN
 F 3 "~" H 6900 2500 50  0001 C CNN
-F 4 "C319849" H 6900 2500 50  0001 C CNN "LCSC"
+F 4 "C488999" H 6900 2500 50  0001 C CNN "LCSC"
 	1    6900 2500
 	1    0    0    -1
@@
 P 7000 2500
 F 0 "R4" H 6950 2700 50  0000 L CNN
-F 1 "7.5K" V 7000 2400 50  0000 L CNN
+F 1 "6.3K" V 7000 2400 50  0000 L CNN
 F 2 "Resistor_SMD:R_1206_3216Metric_Pad1.30x1.75mm_HandSolder" V 6930 2500 50  0001 C CNN
 F 3 "~" H 7000 2500 50  0001 C CNN
-F 4 "C352034" H 7000 2500 50  0001 C CNN "LCSC"
+F 4 "C488915" H 7000 2500 50  0001 C CNN "LCSC"
 	1    7000 2500
 	1    0    0    -1
