File: kicad/mmx-vrm.sch (KiCad schematic (older format))
At the start: 18 parts, among them J1 Conn_02x15_Row_Letter_First, SW1 SW_DIP_x03, U1 LM2596S, U2 LM2596S

Commit message: Revert "Renamed project into s7-vrm"
This reverts commit abb7c84a7e06dd52f3d76b1c246c1366ac80b644.
Parts:
- J1: footprint s7-vrm:EDGE_30-pin -> mmx-vrm:EDGE_30-pin
Changed lines of the file:
@@
 encoding utf-8
 Sheet 1 1
-Title "s7-vrm"
+Title "MMX-VRM"
 Date "2021-11-19"
 Rev "0.2"
@@
 F 0 "J1" H 2700 1967 50  0000 C CNN
 F 1 "Conn_02x15_Row_Letter_First" H 2700 3626 50  0001 C CNN
-F 2 "s7-vrm:EDGE_30-pin" H 2650 2800 50  0001 C CNN
+F 2 "mmx-vrm:EDGE_30-pin" H 2650 2800 50  0001 C CNN
 F 3 "~" H 2650 2800 50  0001 C CNN
 F 4 "C132129" H 2650 2800 50  0001 C CNN "LCSC"

Commit message: First raw version
Parts:
- removed D1, D2: 1N5820, Diode_SMD:D_SMA, symbol Device:D_Schottky
- removed L2: 47uH, Inductor_SMD:L_10.4x10.4_H4.8, symbol Device:L
- removed U1, U2: LM2596S, Package_TO_SOT_SMD:TO-263-5_TabPin3, symbol Regulator_Switching:LM2596S-ADJ
- added C2, C5: 1mF, Capacitor_THT:CP_Radial_D6.3mm_P2.50mm, symbol Device:CP
- added C6, C7: 0.1u, Capacitor_SMD:C_1206_3216Metric_Pad1.33x1.80mm_HandSolder, symbol Device:C
- added C8, C9: C, Capacitor_SMD:C_1206_3216Metric_Pad1.33x1.80mm_HandSolder, symbol Device:C
- added D1: D, Diode_SMD:D_1206_3216Metric_Pad1.42x1.75mm_HandSolder, symbol Device:D
- added Q1, Q2: Q_NMOS_GDS, Package_TO_SOT_SMD:TO-252-2, symbol Device:Q_NMOS_GDS
- added Q3: Q_NPN_BCE, Package_TO_SOT_SMD:SOT-23, symbol Device:Q_NPN_BCE
- added R6: 3K, Resistor_SMD:R_1206_3216Metric_Pad1.30x1.75mm_HandSolder, symbol Device:R
- added R9: R, Resistor_SMD:R_1206_3216Metric_Pad1.30x1.75mm_HandSolder, symbol Device:R
- added U1: NCP1579, Package_SO:SOIC-8_3.9x4.9mm_P1.27mm, symbol mmx-vrm:NCP1579
- C1: renamed from C2; value 820u -> 1mF; footprint Capacitor_THT:CP_Radial_D10.0mm_P5.00mm -> Capacitor_THT:CP_Radial_D6.3mm_P2.50mm; LCSC C442583 -> C494544
- C3: value 10nF -> 0.1u
- C4: renamed from C1; value 820u -> 1mF; footprint Capacitor_THT:CP_Radial_D10.0mm_P5.00mm -> Capacitor_THT:CP_Radial_D6.3mm_P2.50mm; LCSC C442583 -> C494544
- R2: renamed from R6; value 1.6K -> 3K
- R3: value 9.1K -> 21K
- R4: value 6.3K -> 15K
- R5: value 3K -> 6,3K
- SW1: footprint Button_Switch_THT:SW_DIP_SPSTx03_Slide_9.78x9.8mm_W7.62mm_P2.54mm -> Button_Switch_THT:SW_DIP_SPSTx04_Slide_9.78x12.34mm_W7.62mm_P2.54mm; symbol Switch:SW_DIP_x03 -> Switch:SW_DIP_x04
- renumbered R7 to R1, R1 to R7, R2 to R8
Connections:
- wire segments 48 -> 57
- no-connect marks 1 -> 2
Other:
- moved on the sheet: C1, C4, L1, R1, R2, R3, R4, R5, R7, R8

Commit message: Add LCSC IDs and documentation
Parts:
- added C4: 4.7u, Capacitor_SMD:C_1206_3216Metric_Pad1.33x1.80mm_HandSolder, symbol Device:C
- added C8: 0.1u, Capacitor_SMD:C_1206_3216Metric_Pad1.33x1.80mm_HandSolder, symbol Device:C
- added R10: 15K, Resistor_SMD:R_1206_3216Metric_Pad1.30x1.75mm_HandSolder, symbol Device:R
- C10: renamed from C8; value C -> 386p; LCSC (none) -> C577165
- C11: renamed from C7; LCSC C431006 -> C696845
- C3: LCSC C431006 -> C696845
- C7: renamed from C6; value 0.1u -> 4.7u; LCSC C431006 -> C105997
- C9: value C -> 81n; LCSC (none) -> C976248
- D1: LCSC (none) -> C109000
- L1: value 47uH -> 1,2uH; footprint Inductor_SMD:L_10.4x10.4_H4.8 -> Inductor_SMD:L_12x12mm_H4.5mm; LCSC C182153 -> C337553
- Q3: value Q_NPN_BCE -> Q_NPN_BEC; symbol Device:Q_NPN_BCE -> Device:Q_NPN_BEC
- R1, R8: LCSC C406728 -> C144508
- R2: LCSC C204679 -> C229609
- R3: LCSC C706447 -> C229446
- R4: LCSC C488915 -> C144515
- R5: LCSC C132648 -> C229767
- R6: LCSC C132648 -> C229609
- R9: value R -> 3K; LCSC (none) -> C229609
- SW1: value SW_DIP_x03 -> SW_DIP_x04; LCSC C52648 -> C15781
- U1: LCSC (none) -> C235991
- renumbered C4 to C5, C5 to C6
Connections:
- wire segments 57 -> 64
Other:
- moved on the sheet: C1, C10, C11, C2, C3, C5, C6, C7, C9, D1, J1, L1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

Commit message: Minor fixes.
- Changed LCSC part numbers (due to shortage)
- Enlarged GND plane distance
Parts:
- C10: LCSC C577165 -> C2760364
Changed lines of the file:
@@
 F 2 "Capacitor_SMD:C_1206_3216Metric_Pad1.33x1.80mm_HandSolder" H 5588 4100 50  0001 C CNN
 F 3 "~" H 5550 4250 50  0001 C CNN
-F 4 "C577165" H 5550 4250 50  0001 C CNN "LCSC"
+F 4 "C2760364" H 5550 4250 50  0001 C CNN "LCSC"
 	1    5550 4250
 	1    0    0    -1
