File: kicad/s7-vrm.sch (KiCad schematic (older format))
At the start: 18 parts, among them J1 Conn_02x15_Row_Letter_First, SW1 SW_DIP_x03, U1 LM2596S, U2 LM2596S

Commit message: Renamed project into s7-vrm
Parts:
- J1: footprint mmx-vrm:EDGE_30-pin -> s7-vrm:EDGE_30-pin
Changed lines of the file:
@@
 encoding utf-8
 Sheet 1 1
-Title "MMX-VRM"
+Title "s7-vrm"
 Date "2021-11-19"
 Rev "0.2"
@@
 F 0 "J1" H 2700 1967 50  0000 C CNN
 F 1 "Conn_02x15_Row_Letter_First" H 2700 3626 50  0001 C CNN
-F 2 "mmx-vrm:EDGE_30-pin" H 2650 2800 50  0001 C CNN
+F 2 "s7-vrm:EDGE_30-pin" H 2650 2800 50  0001 C CNN
 F 3 "~" H 2650 2800 50  0001 C CNN
 F 4 "C132129" H 2650 2800 50  0001 C CNN "LCSC"

Commit message: Tweaked lower voltages
Parts:
- R3: value 9K -> 9.1K; LCSC C488999 -> C706447
- R5: value 2.9K -> 3K; LCSC C488724 -> C132648
Changed lines of the file:
@@
 P 7100 2500
 F 0 "R5" H 7050 2700 50  0000 L CNN
-F 1 "2.9K" V 7100 2450 50  0000 L CNN
+F 1 "3K" V 7100 2450 50  0000 L CNN
 F 2 "Resistor_SMD:R_1206_3216Metric_Pad1.30x1.75mm_HandSolder" V 7030 2500 50  0001 C CNN
 F 3 "~" H 7100 2500 50  0001 C CNN
-F 4 "C488724" H 7100 2500 50  0001 C CNN "LCSC"
+F 4 "C132648" H 7100 2500 50  0001 C CNN "LCSC"
 	1    7100 2500
 	1    0    0    -1
@@
 P 6900 2500
 F 0 "R3" H 6850 2700 50  0000 L CNN
-F 1 "9K" V 6900 2400 50  0000 L CNN
+F 1 "9.1K" V 6900 2400 50  0000 L CNN
 F 2 "Resistor_SMD:R_1206_3216Metric_Pad1.30x1.75mm_HandSolder" V 6830 2500 50  0001 C CNN
 F 3 "~" H 6900 2500 50  0001 C CNN
-F 4 "C488999" H 6900 2500 50  0001 C CNN "LCSC"
+F 4 "C706447" H 6900 2500 50  0001 C CNN "LCSC"
 	1    6900 2500
 	1    0    0    -1
